Commit message: Sección 4: Digital Twin (no camera yet)

File: ros2_ws/src/arduinobot_description/urdf/arduinobot.urdf.xacro (robot description, xacro)
@@ -3,4 +3,13 @@
     <xacro:property name="effort" value="30.0" />
     <xacro:property name="velocity" value="10.0" />
+    <xacro:macro name="default_inertial" params="mass">
+        <inertial>
+            <mass value="${mass}" />
+            <inertia ixx="1.0" ixy="0.0" ixz="0.0"
+                iyy="1.0" iyz="0.0"
+                izz="1.0"
+            />
+        </inertial>
+    </xacro:macro>
     <link name="world" />
     <link name="base_link">
@@ -12,4 +21,12 @@
             </geometry>
         </visual>
+        <collision>
+            <origin xyz="-0.5 -0.5 0" rpy="0 0 0" />
+            <geometry>
+                <mesh filename="package://arduinobot_description/meshes/basement.STL"
+                    scale="0.01 0.01 0.01" />
+            </geometry>
+        </collision>
+        <xacro:default_inertial mass="1.0" />
     </link>
     <link name="base_plate_link">
@@ -21,4 +38,12 @@
             </geometry>
         </visual>
+        <collision>
+            <origin xyz="-0.39 -0.39 -0.56" rpy="0 0 0" />
+            <geometry>
+                <mesh filename="package://arduinobot_description/meshes/base_plate.STL"
+                    scale="0.01 0.01 0.01" />
+            </geometry>
+        </collision>
+        <xacro:default_inertial mass="0.1" />
     </link>
     <link name="forward_drive_arm_link">
@@ -31,4 +56,13 @@
             <origin xyz="0.19 0.06 0.08" rpy="0 ${-pi / 2.0} ${pi / 2.0}" />
         </visual>
+        <collision>
+            <geometry>
+                <mesh filename="package://arduinobot_description/meshes/forward_drive_arm.STL"
+                    scale="0.01 0.01 0.01"
+                />
+            </geometry>
+            <origin xyz="0.19 0.06 0.08" rpy="0 ${-pi / 2.0} ${pi / 2.0}" />
+        </collision>
+        <xacro:default_inertial mass="0.1" />
     </link>
     <link name="horizontal_arm_link">
@@ -41,4 +75,13 @@
             <origin xyz="-0.03 -0.4 -0.06" rpy="${pi / 2.0} 0 ${pi / 2.0}" />
         </visual>
+        <collision>
+            <geometry>
+                <mesh filename="package://arduinobot_description/meshes/horizontal_arm.STL"
+                    scale="0.01 0.01 0.01"
+                />
+            </geometry>
+            <origin xyz="-0.03 -0.4 -0.06" rpy="${pi / 2.0} 0 ${pi / 2.0}" />
+        </collision>
+        <xacro:default_inertial mass="0.1" />
     </link>
     <link name="claw_support_link">
@@ -51,4 +94,13 @@
             <origin xyz="0 -0.05 -0.15" rpy="0 0 ${pi / 2.0}" />
         </visual>
+        <collision>
+            <geometry>
+                <mesh filename="package://arduinobot_description/meshes/claw_support.STL"
+                    scale="0.01 0.01 0.01"
+                />
+            </geometry>
+            <origin xyz="0 -0.05 -0.15" rpy="0 0 ${pi / 2.0}" />
+        </collision>
+        <xacro:default_inertial mass="0.05" />
     </link>
     <link name="gripper_right_link">
@@ -61,4 +113,13 @@
             <origin xyz="-0.1 0.5 -0.1" rpy="0 0 ${-pi / 2.0}" />
         </visual>
+        <collision>
+            <geometry>
+                <mesh filename="package://arduinobot_description/meshes/right_finger.STL"
+                    scale="0.01 0.01 0.01"
+                />
+            </geometry>
+            <origin xyz="-0.1 0.5 -0.1" rpy="0 0 ${-pi / 2.0}" />
+        </collision>
+        <xacro:default_inertial mass="0.01" />
     </link>
     <link name="gripper_left_link">
@@ -71,4 +132,13 @@
             <origin xyz="-0.04 0.5 -0.1" rpy="0 0 ${-pi / 2.0}" />
         </visual>
+        <collision>
+            <geometry>
+                <mesh filename="package://arduinobot_description/meshes/left_finger.STL"
+                    scale="0.01 0.01 0.01"
+                />
+            </geometry>
+            <origin xyz="-0.04 0.5 -0.1" rpy="0 0 ${-pi / 2.0}" />
+        </collision>
+        <xacro:default_inertial mass="0.01" />
     </link>
     <link name="rgb_camera_link">
@@ -81,4 +151,13 @@
             <origin xyz="-0.1 0.125 0.15" rpy="${-pi / 2.0} 0 ${-pi / 2.0}" />
         </visual>
+        <collision>
+            <geometry>
+                <mesh filename="package://arduinobot_description/meshes/pi_camera.STL"
+                    scale="0.01 0.01 0.01"
+                />
+            </geometry>
+            <origin xyz="-0.1 0.125 0.15" rpy="${-pi / 2.0} 0 ${-pi / 2.0}" />
+        </collision>
+        <xacro:default_inertial mass="0.001" />
     </link>
     <joint name="world__base_joint" type="fixed">
@@ -133,3 +212,81 @@
         <origin xyz="0 0.45 0.2" rpy="0 -0.5 1.57" />
     </joint>
+    <gazebo>
+        <plugin name="joint_state_publisher" filename="libgazebo_ros_joint_state_publisher.so">
+            <jointName>
+                base__base_plate_joint,base_plate__forward_drive_arm_joint,horizontal_arm__base_plate_forward_drive_arm_joint,claw_support__gripper_right_joint,claw_support_link__gripper_left_joint</jointName>
+        </plugin>
+    </gazebo>
+    <!-- <gazebo reference="rgb_camera_link">
+        <sensor name="rgb_camera" type="camera">
+            <always_on>true</always_on>
+            <update_rate>30.0</update_rate>
+            <visualize>true</visualize>
+            <topic>image_raw</topic>
+            <gz_frame_id>rgb_camera_link</gz_frame_id>
+            <camera name="camera">
+                <horizontal_fov>1.21126</horizontal_fov>
+                <image>
+                    <width>2304</width>
+                    <height>1296</height>
+                    <format>R8G8B8</format>
+                </image>
+                <distortion>
+                    <k1>0.0</k1>
+                    <k2>0.0</k2>
+                    <k3>0.0</k3>
+                    <p1>0.0</p1>
+                    <p2>0.0</p2>
+                    <center>0.5 0.5</center>
+                </distortion>
+            </camera>
+            <plugin name="camera_controller" filename="libgazebo_ros_camera.so">
+                <imageTopicName>image_raw</imageTopicName>
+                <cameraInfoTopicName>camera_info</cameraInfoTopicName>
+                <gz_frame_id>rgb_camera_link</gz_frame_id>
+                <frameName>rgb_camera_link</frameName>
+            </plugin>
+        </sensor>
+    </gazebo> -->
+    <!-- camera -->
+  <gazebo reference="rgb_camera_link">
+    <sensor type="camera" name="camera1">
+      <update_rate>30.0</update_rate>
+      <camera name="camera1">
+        <horizontal_fov>1.3962634</horizontal_fov>
+        <image>
+          <width>800</width>
+          <height>800</height>
+          <format>R8G8B8</format>
+        </image>
+        <clip>
+          <near>0.02</near>
+          <far>300</far>
+        </clip>
+        <noise>
+          <type>gaussian</type>
+          <!-- Noise is sampled independently per pixel on each frame.
+               That pixel's noise value is added to each of its color
+               channels, which at that point lie in the range [0,1]. -->
+          <mean>0.0</mean>
+          <stddev>0.007</stddev>
+        </noise>
+      </camera>
+      <plugin name="camera_controller" filename="libgazebo_ros_camera.so">
+        <alwaysOn>true</alwaysOn>
+        <updateRate>0.0</updateRate>
+        <cameraName>camera1</cameraName>
+        <imageTopicName>image_raw</imageTopicName>
+        <cameraInfoTopicName>camera_info</cameraInfoTopicName>
+        <gz_frame_id>/rgb_camera_link</gz_frame_id>
+        <frameName>rgb_camera_link</frameName>
+        <hackBaseline>0.07</hackBaseline>
+        <distortionK1>0.0</distortionK1>
+        <distortionK2>0.0</distortionK2>
+        <distortionK3>0.0</distortionK3>
+        <distortionT1>0.0</distortionT1>
+        <distortionT2>0.0</distortionT2>
+      </plugin>
+    </sensor>
+  </gazebo>
 </robot>

Commit message: Sección 5: Control

File: ros2_ws/src/arduinobot_description/urdf/arduinobot.urdf.xacro (robot description, xacro)
@@ -1,4 +1,9 @@
 <?xml version="1.0"?>
 <robot xmlns:xacro="http://www.ros.org/wiki/xacro" name="ardduinobot">
+    <!-- For use plugin in a specific ROS2 version -->
+    <xacro:arg name="is_ignition" default="true" />
+    <xacro:include filename="$(find arduinobot_description)/urdf/arduinobot_gazebo.xacro" />
+    <xacro:include filename="$(find arduinobot_description)/urdf/arduinobot_ros2_control.xacro" />
+    <xacro:include filename="$(find arduinobot_description)/urdf/material.xacro" />
     <xacro:property name="effort" value="30.0" />
     <xacro:property name="velocity" value="10.0" />
@@ -20,4 +25,5 @@
                     scale="0.01 0.01 0.01" />
             </geometry>
+            <material name="blue" />
         </visual>
         <collision>
@@ -37,4 +43,5 @@
                     scale="0.01 0.01 0.01" />
             </geometry>
+            <material name="red" />
         </visual>
         <collision>
@@ -54,5 +61,6 @@
                 />
             </geometry>
-            <origin xyz="0.19 0.06 0.08" rpy="0 ${-pi / 2.0} ${pi / 2.0}" />
+            <origin xyz="0.19 0.06 -0.08" rpy="0 ${-pi / 2.0} ${pi / 2.0}" />
+            <material name="green" />
         </visual>
         <collision>
@@ -62,5 +70,5 @@
                 />
             </geometry>
-            <origin xyz="0.19 0.06 0.08" rpy="0 ${-pi / 2.0} ${pi / 2.0}" />
+            <origin xyz="0.19 0.06 -0.08" rpy="0 ${-pi / 2.0} ${pi / 2.0}" />
         </collision>
         <xacro:default_inertial mass="0.1" />
@@ -74,4 +82,5 @@
             </geometry>
             <origin xyz="-0.03 -0.4 -0.06" rpy="${pi / 2.0} 0 ${pi / 2.0}" />
+            <material name="orange" />
         </visual>
         <collision>
@@ -93,4 +102,5 @@
             </geometry>
             <origin xyz="0 -0.05 -0.15" rpy="0 0 ${pi / 2.0}" />
+            <material name="purple" />
         </visual>
         <collision>
@@ -112,4 +122,5 @@
             </geometry>
             <origin xyz="-0.1 0.5 -0.1" rpy="0 0 ${-pi / 2.0}" />
+            <material name="cyan" />
         </visual>
         <collision>
@@ -131,4 +142,5 @@
             </geometry>
             <origin xyz="-0.04 0.5 -0.1" rpy="0 0 ${-pi / 2.0}" />
+            <material name="cyan" />
         </visual>
         <collision>
@@ -150,4 +162,5 @@
             </geometry>
             <origin xyz="-0.1 0.125 0.15" rpy="${-pi / 2.0} 0 ${-pi / 2.0}" />
+            <material name="yellow" />
         </visual>
         <collision>
@@ -166,4 +179,5 @@
         <origin xyz="0 0 0" rpy="0 0 0" />
     </joint>
+    <!-- Joint 1 -->
     <joint name="base__base_plate_joint" type="revolute">
         <parent link="base_link" />
@@ -173,4 +187,5 @@
         <origin xyz="0 0 0.307" rpy="0 0 0" />
     </joint>
+    <!-- Joint 2 -->
     <joint name="base_plate__forward_drive_arm_joint" type="revolute">
         <parent link="base_plate_link" />
@@ -180,4 +195,5 @@
         <origin xyz="-0.02 0 0.35" rpy="0 0 0" />
     </joint>
+    <!-- Joint 3 -->
     <joint name="horizontal_arm__base_plate_forward_drive_arm_joint" type="revolute">
         <parent link="forward_drive_arm_link" />
@@ -192,4 +208,5 @@
         <origin xyz="0 0.82 0" rpy="0 0 0" />
     </joint>
+    <!-- Joint 4 -->
     <joint name="claw_support__gripper_right_joint" type="revolute">
         <parent link="claw_support_link" />
@@ -199,4 +216,5 @@
         <origin xyz="-0.04 0.13 -0.1" rpy="0 0 0" />
     </joint>
+    <!-- Joint 5 -->
     <joint name="claw_support_link__gripper_left_joint" type="revolute">
         <parent link="claw_support_link" />
@@ -250,43 +268,43 @@
     </gazebo> -->
     <!-- camera -->
-  <gazebo reference="rgb_camera_link">
-    <sensor type="camera" name="camera1">
-      <update_rate>30.0</update_rate>
-      <camera name="camera1">
-        <horizontal_fov>1.3962634</horizontal_fov>
-        <image>
-          <width>800</width>
-          <height>800</height>
-          <format>R8G8B8</format>
-        </image>
-        <clip>
-          <near>0.02</near>
-          <far>300</far>
-        </clip>
-        <noise>
-          <type>gaussian</type>
-          <!-- Noise is sampled independently per pixel on each frame.
+    <gazebo reference="rgb_camera_link">
+        <sensor type="camera" name="camera1">
+            <update_rate>30.0</update_rate>
+            <camera name="camera1">
+                <horizontal_fov>1.3962634</horizontal_fov>
+                <image>
+                    <width>800</width>
+                    <height>800</height>
+                    <format>R8G8B8</format>
+                </image>
+                <clip>
+                    <near>0.02</near>
+                    <far>300</far>
+                </clip>
+                <noise>
+                    <type>gaussian</type>
+                    <!-- Noise is sampled independently per pixel on each frame.
                That pixel's noise value is added to each of its color
                channels, which at that point lie in the range [0,1]. -->
-          <mean>0.0</mean>
-          <stddev>0.007</stddev>
-        </noise>
-      </camera>
-      <plugin name="camera_controller" filename="libgazebo_ros_camera.so">
-        <alwaysOn>true</alwaysOn>
-        <updateRate>0.0</updateRate>
-        <cameraName>camera1</cameraName>
-        <imageTopicName>image_raw</imageTopicName>
-        <cameraInfoTopicName>camera_info</cameraInfoTopicName>
-        <gz_frame_id>/rgb_camera_link</gz_frame_id>
-        <frameName>rgb_camera_link</frameName>
-        <hackBaseline>0.07</hackBaseline>
-        <distortionK1>0.0</distortionK1>
-        <distortionK2>0.0</distortionK2>
-        <distortionK3>0.0</distortionK3>
-        <distortionT1>0.0</distortionT1>
-        <distortionT2>0.0</distortionT2>
-      </plugin>
-    </sensor>
-  </gazebo>
+                    <mean>0.0</mean>
+                    <stddev>0.007</stddev>
+                </noise>
+            </camera>
+            <plugin name="camera_controller" filename="libgazebo_ros_camera.so">
+                <alwaysOn>true</alwaysOn>
+                <updateRate>0.0</updateRate>
+                <cameraName>camera1</cameraName>
+                <imageTopicName>image_raw</imageTopicName>
+                <cameraInfoTopicName>camera_info</cameraInfoTopicName>
+                <gz_frame_id>/rgb_camera_link</gz_frame_id>
+                <frameName>rgb_camera_link</frameName>
+                <hackBaseline>0.07</hackBaseline>
+                <distortionK1>0.0</distortionK1>
+                <distortionK2>0.0</distortionK2>
+                <distortionK3>0.0</distortionK3>
+                <distortionT1>0.0</distortionT1>
+                <distortionT2>0.0</distortionT2>
+            </plugin>
+        </sensor>
+    </gazebo>
 </robot>
